Commit message: working articulated body on simple arm

File: Samples~/ZeroSimSamples/Assets/ZeroSimAssets/SimpleRobotArm_ArticulatedBody.urdf (robot description, URDF)
Before this commit: robot SimpleRobotArm_ArticulatedBody, 4 links, 3 joints
Joints:
- joint joint.articulated_body.fixedjoint_from_hand: limit effort=3.40282347e+38 velocity=0.0 -> effort=3.40282347e+38 velocity=100.0; origin xyz=0.0 -0.0 0.300000048 rpy=-0.0 0.0 -0.0 -> xyz=0.0 -0.0 0.29999996399999995 rpy=-0.0 0.0 -0.0
- joint joint.articulated_body.revolutejoint_from_elbow: limit effort=3.40282347e+38 velocity=0.0 -> effort=3.40282347e+38 velocity=100.0; origin xyz=0.0 -0.0 0.30000000600000004 rpy=-0.0 0.0 -0.0 -> xyz=0.0 -0.0 0.3000000718 rpy=-0.0 0.0 -0.0
- joint joint.articulated_body.revolutejoint_from_shoulder: limit effort=3.40282347e+38 velocity=0.0 -> effort=3.40282347e+38 velocity=100.0; origin xyz=0.0 -0.0 0.099999994 rpy=-0.0 0.0 -0.0 -> xyz=0.0 -0.0 0.0999999642 rpy=-0.0 0.0 -0.0
