Commit message: working UR10!

File: Samples~/ZeroSimSamples/Assets/ZeroSimAssets/UR10_rigged.urdf (robot description, URDF)
Before this commit: robot UR10_rigged, 9 links, 6 joints
Links:
- removed link base_pivot
- removed link shoulder_lift
- removed link shoulder_pan
- added link shoulder; visual box size=0.06345073 0.0599891022 0.06847392; visual box size=0.075 0.075 0.2303
- added link shoulder_base; visual box size=0.08861007 0.07516342 0.0805922151
- link base: geometry visual box size=0.08355 0.075 0.019
Joints:
- joint elbow_joint: axis -0.99999994 -5.96046448e-08 0.0 -> 1.0 -0.0 0.0; child shoulder_lift -> elbow; limit effort=3.40282347e+38 velocity=100000.0 -> effort=10.0 velocity=100.0; origin xyz=-0.010000000000000009 -0.0 0.610000014 rpy=-0.0 0.0 -0.0 -> xyz=-0.022499999999999992 -0.0 0.619999979 rpy=-0.0 0.0 -0.0; parent shoulder_pan -> shoulder
- joint shoulder_lift_joint: axis -0.9999999 -1.1920929e-07 0.0 -> -1.0 -0.0 0.0; child shoulder_pan -> shoulder; limit effort=3.40282347e+38 velocity=100000.0 -> effort=10.0 velocity=100.0; origin xyz=-0.09 -0.0 0.128000021 rpy=-0.0 0.0 -0.0 -> xyz=-0.0855 -0.0 0.0915000439 rpy=-0.0 0.0 -0.0; parent base_pivot -> shoulder_base
- joint shoulder_pan_joint: axis 0.0 -5.96046448e-08 0.99999994 -> 0.0 -0.0 1.0; child base_pivot -> shoulder_base; limit effort=3.40282347e+38 velocity=100000.0 -> effort=10.0 velocity=100.0; origin xyz=0.0 -0.0 0.0 rpy=-0.0 0.0 -0.0 -> xyz=0.0 -0.0 0.0364999771 rpy=-0.0 0.0 -0.0
- joint wrist_1_joint: axis 0.99999994 -5.96046448e-08 0.0 -> -2.0 -0.0 0.0; child elbow -> wrist-1; limit effort=3.40282347e+38 velocity=100000.0 -> effort=10.0 velocity=100.0; origin xyz=-0.009960235999999997 0.0100000147 0.576400515 rpy=-0.0 0.0 -0.0 -> xyz=-0.0038402560000000002 0.0100000147 0.5644004600000001 rpy=-0.0 0.0 -0.0; parent shoulder_lift -> elbow
- joint wrist_2_joint: axis -0.99999994 -5.96046448e-08 0.0 -> 0.0 -0.0 1.0; child wrist-1 -> wrist-2; limit effort=3.40282347e+38 velocity=100000.0 -> effort=10.0 velocity=100.0; origin xyz=0.0042696450000000025 -0.010000012837354851 -0.002100229999999925 rpy=-0.0 0.0 -0.0 -> xyz=-0.05385033 -0.010000012837354851 0.06189990000000001 rpy=-0.0 0.0 -0.0; parent elbow -> wrist-1
- joint wrist_3_joint: axis -0.99999994 -5.96046448e-08 0.0 -> 0.0 -1.4715822136062044e-15 1.0000000000000002; child wrist-2 -> wrist-3; limit effort=3.40282347e+38 velocity=100000.0 -> effort=10.0 velocity=100.0; origin xyz=-0.12019977700000001 -2.79396775e-09 0.11249995999999984 rpy=-0.0 0.0 -0.0 -> xyz=-0.06019978200000001 -0.0 0.05550002999999992 rpy=1.471582213606204e-15 1.5707963267948963 1.4715822136062052e-15; parent wrist-1 -> wrist-2

Commit message: can now see arm in rviz but still cannot move it in 0sim

File: Samples~/ZeroSimSamples/Assets/ZeroSimAssets/UR10_rigged.urdf (robot description, URDF)
Before this commit: robot UR10_rigged, 8 links, 6 joints
Links:
- removed link base
- removed link elbow
- removed link shoulder
- removed link shoulder_base
- removed link tool-flange-occurrence
- removed link wrist-1
- removed link wrist-2
- removed link wrist-3
- added link base_link; visual box size=0.08355 0.075 0.019
- added link ee_link; visual box size=0.04505 0.04499998 0.01525
- added link forearm_link; visual box size=0.0499491356 0.0454888642 0.05938407; visual box size=0.058 0.225649983 0.058
- added link shoulder_link; visual box size=0.08861007 0.07516342 0.0805922151
- added link upper_arm_link; visual box size=0.06345073 0.0599891022 0.06847392; visual box size=0.075 0.075 0.2303
- added link wrist_1_link; visual box size=0.0499491356 0.0454888642 0.05938407
- added link wrist_2_link; visual box size=0.0499491356 0.0454888642 0.05938407
- added link wrist_3_link
Joints:
- added joint ee_fixed_joint: type fixed, parent wrist_3_link, child ee_link, origin xyz=-0.005500231999999994 4.65661285e-09 -0.001800299999999977 rpy=3.5527128400000008e-15 0.0 -0.0
- added joint joint.fixed_from_base_link: type fixed, parent base_link, child world, origin xyz=0 0 0 rpy=0 0 0
- joint elbow_joint: child elbow -> forearm_link; limit effort=10.0 velocity=100.0 -> effort=10.0 velocity=500.0; parent shoulder -> upper_arm_link
- joint shoulder_lift_joint: child shoulder -> upper_arm_link; limit effort=10.0 velocity=100.0 -> effort=10.0 velocity=500.0; parent shoulder_base -> shoulder_link
- joint shoulder_pan_joint: child shoulder_base -> shoulder_link; limit effort=10.0 velocity=100.0 -> effort=10.0 velocity=500.0; parent base -> base_link
- joint wrist_1_joint: child wrist-1 -> wrist_1_link; limit effort=10.0 velocity=100.0 -> effort=10.0 velocity=500.0; parent elbow -> forearm_link
- joint wrist_2_joint: child wrist-2 -> wrist_2_link; limit effort=10.0 velocity=100.0 -> effort=10.0 velocity=500.0; parent wrist-1 -> wrist_1_link
- joint wrist_3_joint: child wrist-3 -> wrist_3_link; limit effort=10.0 velocity=100.0 -> effort=10.0 velocity=500.0; parent wrist-2 -> wrist_2_link

Commit message: can "see" ur10 in rviz (very broken)

File: Samples~/ZeroSimSamples/Assets/ZeroSimAssets/UR10_rigged.urdf (robot description, URDF)
Before this commit: robot UR10_rigged, 8 links, 8 joints
Joints:
- removed joint joint.fixed_from_base_link

Commit message: working moveit!  (some bugs but it works!)

File: Samples~/ZeroSimSamples/Assets/ZeroSimAssets/UR10_rigged.urdf (robot description, URDF)
Before this commit: robot UR10_rigged, 8 links, 7 joints
Links:
- added link world
Joints:
- added joint world_to_baselink: type fixed, parent world, child base_link, origin xyz=0.0 0.0 0.0 rpy=0.0 0.0 -0.0
